File: kicad/PSN_TRX.kicad_pcb (KiCad board)
At the start: 4 copper layers, 134 x 129.6 mm, 282 parts, among them IC1 R-78E5.0-1.0, IC2 NJM2904, J1 RF_IN, J10 MIC-IN, J11 AE-ADS1015, J2 PWR_IN, J3 TX-ON-LED, J4 Volume, J5 Volume, J6 SP-OUT, J7 Encoder, J8 NX4832T035, J9 I2C_OUT-LCD, K1 G5V-2 DC12, Q1 2SA1015, Q10 2SK439, Q11 2SK439, Q12 2SC1815, Q13 2SC2120, Q14 2SA950, Q15 2SC1815, Q16 2SC1815, Q17 2SC1815, Q18 2SC1815, Q19 2SC1815, Q2 3SK59, Q20 J310, Q21 2SC1815, Q22 2SC1815, Q23 2SC1815, Q25 J310, Q3 RD06HVF1, Q4 J310, Q5 J310, Q6 2SC1815, Q8 2SC1815, Q9 2SC1815, U1 Si5351_DIP8, U2 LP2950-3.3_TO92, U3 Seeeduino_XIAO_Socket, U4 NJM2594V, U5 NJM2594V, U6 78L05, U7 AD8307ANZ, Y1 12MHz, Y2 12MHz, Y3 12MHz, Y4 12MHz, Y5 12MHz, Y6 12MHz

Commit message: 受信の JFET 4 個（Q4・Q5・Q20・Q25）を J310 から 2SK192A-GR に置き換え
- 2SK192A（東芝）はピン 1 D・2 S・3 G で J310 と同じ並び。TO-92_Inline のまま、基板のパターン・配置は変更なし
- R66（Q20 のソース）100Ω → 47Ω。R5 は 3SK59 用の 120Ω のまま、Q4・Q5 を付けるときは 47Ω（22〜100Ω で 5〜8mA）
- DRC 0・未配線 0・回路図との不一致 0、ERC 未除外 0。ガーバーは部品の値を含まないので出し直しなし
- 部品表（bom・購入用・まとめ・BOM.md・JLCPCB BOM・座標ファイル）、README、調整手順、JLCPCB 提出資料、部品実装図 PDF を更新
- シミュレーション: 2SK192A-GR の模型（Vp −2V・IDSS 10mA、個体差 −1.2〜−3V・6〜14mA）。RF 増幅の利得 +10.9 → +7.7dB、前段 NF 0.95dB、AGC の幅 16.1dB
- ファームウェア: RSSI_S9_MV 1900 → 1830、AGC_TARGET_MV 1750 → 1680（S9 で AD8307 の入力 −8.1 → −10.9dBm）

Co-Authored-By: Claude Opus 5.5 <noreply@anthropic.com>
Parts:
- Q20, Q25, Q4, Q5: value J310 -> 2SK192A
- R66: value 100 -> 47
Changed lines of the file:
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@@
 			)
 		)
-		(property "Value" "J310"
+		(property "Value" "2SK192A"
 			(at 1.27 2.79 270)
 			(layer "F.Fab")
@@
 			)
 		)
-		(property "Description" "RF 増幅のカスコード下段（ソース接地）。V2 改: 2N3819 → J310（TO-92、1 D・2 S・3 G）"
+		(property "Description" "RF 増幅のカスコード下段（ソース接地）。V2 改: 2N3819 → J310 → 2SK192A-GR（TO-92、1 D・2 S・3 G）"
 			(at 0 0 270)
 			(unlocked yes)
@@
 			)
 		)
-		(property "Description" "Q2（3SK59 / J310 カスコード）のドレイン負荷。C11 33p と 12MHz に同調"
+		(property "Description" "Q2（3SK59 / 2SK192A-GR カスコード）のドレイン負荷。C11 33p と 12MHz に同調"
 			(at 0 0 180)
 			(layer "F.Fab")
@@
 			)
 		)
-		(property "Value" "J310"
+		(property "Value" "2SK192A"
 			(at 1.27 2.79 270)
 			(layer "F.Fab")
@@
 			)
 		)
-		(property "Description" "RF 増幅のカスコード上段。ゲートは R95 で AGC（Q2_G2）へ。RF 段にも AGC・RF ゲインが効く"
+		(property "Description" "RF 増幅のカスコード上段。ゲートは R95 で AGC（Q2_G2）へ。RF 段にも AGC・RF ゲインが効く。2SK192A-GR"
 			(at 0 0 270)
 			(unlocked yes)
@@
 			)
 		)
-		(property "Value" "100"
+		(property "Value" "47"
 			(at 1.27 2.37 90)
 			(layer "F.Fab")
@@
 			)
 		)
-		(property "Description" "カスコード下段のソース抵抗（Id 約 12mA）"
+		(property "Description" "カスコード下段 Q20（2SK192A-GR）のソース抵抗（Id 約 6〜8mA）"
 			(at 0 0 90)
 			(layer "F.Fab")
@@
 			)
 		)
-		(property "Description" ""
+		(property "Description" "Q2 のソース抵抗（3SK59 は 120Ω）。Q4・Q5（2SK192A-GR）を付けるときは 47Ω にし、22〜100Ω で 5〜8mA に合わせる"
 			(at 0 0 0)
 			(layer "F.Fab")
@@
 			)
 		)
-		(property "Value" "J310"
+		(property "Value" "2SK192A"
 			(at 1.27 2.79 180)
 			(layer "F.Fab")
@@
 			)
 		)
-		(property "Description" "N-Channel JFET J310（TO-92、1 D・2 S・3 G。買った品のデータシートでピン配置を確認）"
+		(property "Description" "IF 増幅のカスコード上段（Q2 の代わり）。N-Channel JFET 2SK192A（GR ランク、IDSS 6〜14mA。東芝 TO-92 小型 2-4E1D、1 D・2 S・3 G）"
 			(at 0 0 180)
 			(unlocked yes)
@@
 			)
 		)
-		(property "Value" "J310"
+		(property "Value" "2SK192A"
 			(at 1.27 2.79 0)
 			(layer "F.Fab")
@@
 			)
 		)
-		(property "Description" "N-Channel JFET J310（TO-92、1 D・2 S・3 G。買った品のデータシートでピン配置を確認）"
+		(property "Description" "IF 増幅のカスコード下段（Q2 の代わり）。R5 は 47Ω に。N-Channel JFET 2SK192A（GR ランク、IDSS 6〜14mA。東芝 TO-92 小型 2-4E1D、1 D・2 S・3 G）"
 			(at 0 0 0)
 			(unlocked yes)
