File: kicad/PSN_TRX.kicad_pcb (KiCad board)
At the start: 4 copper layers, 134 x 129.6 mm, 282 parts, among them IC1 R-78E5.0-1.0, IC2 NJM2904, J1 RF_IN, J10 MIC-IN, J11 AE-ADS1015, J2 PWR_IN, J3 TX-ON-LED, J4 Volume, J5 Volume, J6 SP-OUT, J7 Encoder, J8 NX4832T035, J9 I2C_OUT-LCD, K1 G5V-2 DC12, Q1 2SA1015, Q10 2SK439, Q11 2SK439, Q12 2SC1815, Q13 2SC2120, Q14 2SA950, Q15 2SC1815, Q16 2SC1815, Q17 2SC1815, Q18 2SC1815, Q19 2SC1815, Q2 3SK59, Q20 2SK192A, Q21 2SC1815, Q22 2SC1815, Q23 2SC1815, Q25 2SK192A, Q3 RD06HVF1, Q4 2SK192A, Q5 2SK192A, Q6 2SC1815, Q8 2SC1815, Q9 2SC1815, U1 Si5351_DIP8, U2 LP2950-3.3_TO92, U3 Seeeduino_XIAO_Socket, U4 NJM2594V, U5 NJM2594V, U6 78L05, U7 AD8307ANZ, Y1 12MHz, Y2 12MHz, Y3 12MHz, Y4 12MHz, Y5 12MHz, Y6 12MHz

Commit message: L19 のタップを +9V 側から 2 回目 → 3 回目に（2SK192A-GR で下がった利得を戻す）
- L19 の値を T30-6 11T/3T に（L18 は 11T/2T のまま）。基板は変更なし（DRC 0・未配線 0・回路図との不一致 0、ERC 0）
- シミュレーション: RF 増幅 +7.7 → +10.5dB、前段の電力利得 +19.9dB・雑音指数 0.96dB、全体の雑音指数 1.3dB（混合器 NF 10dB）
- S9 で AD8307 の入力 −8.2dBm（J310 のときと同じ）なので、ファームウェアの RSSI_S9_MV 1900・AGC_TARGET_MV 1750 に戻す
- 部品表（L18・L19 を別の行に）、JLCPCB BOM・座標ファイル、README、調整手順、提出資料、部品実装図 PDF を更新

Co-Authored-By: Claude Opus 5.5 <noreply@anthropic.com>
Parts:
- L19: value T30-6 11T/2T -> T30-6 11T/3T
Changed lines of the file:
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@@
 			)
 		)
-		(property "Value" "T30-6 11T/2T"
+		(property "Value" "T30-6 11T/3T"
 			(at 2.54 5.2 90)
 			(layer "F.Fab")
@@
 			)
 		)
-		(property "Description" "RF 増幅の出力同調（ドレイン = 1 番、+9V = 3 番、タップ 2 番から混合器へ）"
+		(property "Description" "RF 増幅の出力同調（ドレイン = 1 番、+9V = 3 番、+9V 側から 3 回目のタップ 2 番から混合器へ）"
 			(at 0 0 90)
 			(layer "F.Fab")
