File: kicad/PSN_TRX.kicad_sch (KiCad schematic)
At the start: 280 parts, among them IC1 R-78E5.0-1.0, IC2 NJM2904, J1 RF_IN, J10 MIC-IN, J11 AE-ADS1015, J2 PWR_IN, J3 TX-ON-LED, J4 Volume, J5 Volume, J6 SP-OUT, J7 Encoder, J8 NX4832T035, J9 I2C_OUT-LCD, K1 G5V-2 DC12, Q1 2SA1015, Q10 2SK439, Q11 2SK439, Q12 2SC1815, Q13 2SC2120, Q14 2SA950, Q15 2SC1815, Q16 2SC1815, Q17 2SC1815, Q18 2SC1815, Q19 2SC1815, Q2 3SK59, Q20 J310, Q21 2SC1815, Q22 2SC1815, Q23 2SC1815, Q25 J310, Q3 RD06HVF1, Q4 J310, Q5 J310, Q6 2SC1815, Q8 2SC1815, Q9 2SC1815, U1 Si5351_DIP8, U2 LP2950-3.3_TO92, U3 Seeeduino_XIAO_Socket, U4 NJM2594V, U5 NJM2594V, U6 78L05, U7 AD8307ANZ, Y1 12MHz, Y2 12MHz, Y3 12MHz, Y4 12MHz, Y5 12MHz, Y6 12MHz

Commit message: 受信の JFET 4 個（Q4・Q5・Q20・Q25）を J310 から 2SK192A-GR に置き換え
- 2SK192A（東芝）はピン 1 D・2 S・3 G で J310 と同じ並び。TO-92_Inline のまま、基板のパターン・配置は変更なし
- R66（Q20 のソース）100Ω → 47Ω。R5 は 3SK59 用の 120Ω のまま、Q4・Q5 を付けるときは 47Ω（22〜100Ω で 5〜8mA）
- DRC 0・未配線 0・回路図との不一致 0、ERC 未除外 0。ガーバーは部品の値を含まないので出し直しなし
- 部品表（bom・購入用・まとめ・BOM.md・JLCPCB BOM・座標ファイル）、README、調整手順、JLCPCB 提出資料、部品実装図 PDF を更新
- シミュレーション: 2SK192A-GR の模型（Vp −2V・IDSS 10mA、個体差 −1.2〜−3V・6〜14mA）。RF 増幅の利得 +10.9 → +7.7dB、前段 NF 0.95dB、AGC の幅 16.1dB
- ファームウェア: RSSI_S9_MV 1900 → 1830、AGC_TARGET_MV 1750 → 1680（S9 で AD8307 の入力 −8.1 → −10.9dBm）

Co-Authored-By: Claude Opus 5.5 <noreply@anthropic.com>
Parts:
- Q20, Q25, Q4, Q5: value J310 -> 2SK192A
- R66: value 100 -> 47
Other:
- note added: "L18（入力同調）→ 2SK192A-GR カスコード（Q20・Q25）→ L19（出力同調）。RF 段にも AGC・RF ゲインが効く"
- note added: "Q4・Q5（2SK192A-GR カスコード）は Q2（3SK59）の代わり。どちらか一方を付ける。R5 は 47Ω に"
- note removed: "L18（入力同調）→ J310 カスコード（Q20・Q25）→ L19（出力同調）。RF 段にも AGC・RF ゲインが効く"
- note removed: "Q4・Q5（J310 カスコード）は Q2（3SK59）の代わり。どちらか一方を付ける"
Changed lines of the file:
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@@
 		)
 	)
-	(text "Q4・Q5（J310 カスコード）は Q2（3SK59）の代わり。どちらか一方を付ける"
+	(text "Q4・Q5（2SK192A-GR カスコード）は Q2（3SK59）の代わり。どちらか一方を付ける。R5 は 47Ω に"
 		(exclude_from_sim no)
 		(at 529.59 200.66 0)
@@
 		)
 	)
-	(text "L18（入力同調）→ J310 カスコード（Q20・Q25）→ L19（出力同調）。RF 段にも AGC・RF ゲインが効く"
+	(text "L18（入力同調）→ 2SK192A-GR カスコード（Q20・Q25）→ L19（出力同調）。RF 段にも AGC・RF ゲインが効く"
 		(exclude_from_sim no)
 		(at 121.92 104.14 0)
@@
 			)
 		)
-		(property "Value" "J310"
+		(property "Value" "2SK192A"
 			(at 226.06 130.81 0)
 			(show_name no)
@@
 			)
 		)
-		(property "Description" "RF 増幅のカスコード上段。ゲートは R95 で AGC（Q2_G2）へ。RF 段にも AGC・RF ゲインが効く"
+		(property "Description" "RF 増幅のカスコード上段。ゲートは R95 で AGC（Q2_G2）へ。RF 段にも AGC・RF ゲインが効く。2SK192A-GR"
 			(at 220.98 129.54 0)
 			(hide yes)
@@
 			)
 		)
-		(property "Value" "J310"
+		(property "Value" "2SK192A"
 			(at 226.06 148.59 0)
 			(show_name no)
@@
 			)
 		)
-		(property "Description" "RF 増幅のカスコード下段（ソース接地）。V2 改: 2N3819 → J310（TO-92、1 D・2 S・3 G）"
+		(property "Description" "RF 増幅のカスコード下段（ソース接地）。V2 改: 2N3819 → J310 → 2SK192A-GR（TO-92、1 D・2 S・3 G）"
 			(at 220.98 147.32 0)
 			(hide yes)
@@
 			)
 		)
-		(property "Description" ""
+		(property "Description" "Q2 のソース抵抗（3SK59 は 120Ω）。Q4・Q5（2SK192A-GR）を付けるときは 47Ω にし、22〜100Ω で 5〜8mA に合わせる"
 			(at 618.49 143.51 0)
 			(hide yes)
@@
 			)
 		)
-		(property "Description" "Q2（3SK59 / J310 カスコード）のドレイン負荷。C11 33p と 12MHz に同調"
+		(property "Description" "Q2（3SK59 / 2SK192A-GR カスコード）のドレイン負荷。C11 33p と 12MHz に同調"
 			(at 623.57 120.65 0)
 			(hide yes)
@@
 			)
 		)
-		(property "Value" "100"
+		(property "Value" "47"
 			(at 226.06 157.48 0)
 			(show_name no)
@@
 			)
 		)
-		(property "Description" "カスコード下段のソース抵抗（Id 約 12mA）"
+		(property "Description" "カスコード下段 Q20（2SK192A-GR）のソース抵抗（Id 約 6〜8mA）"
 			(at 223.52 156.21 0)
 			(hide yes)
@@
 			)
 		)
-		(property "Value" "J310"
+		(property "Value" "2SK192A"
 			(at 554.99 168.91 0)
 			(show_name no)
@@
 			)
 		)
-		(property "Description" "N-Channel JFET J310（TO-92、1 D・2 S・3 G。買った品のデータシートでピン配置を確認）"
+		(property "Description" "IF 増幅のカスコード上段（Q2 の代わり）。N-Channel JFET 2SK192A（GR ランク、IDSS 6〜14mA。東芝 TO-92 小型 2-4E1D、1 D・2 S・3 G）"
 			(at 549.91 167.64 0)
 			(hide yes)
@@
 			)
 		)
-		(property "Value" "J310"
+		(property "Value" "2SK192A"
 			(at 554.99 181.61 0)
 			(show_name no)
@@
 			)
 		)
-		(property "Description" "N-Channel JFET J310（TO-92、1 D・2 S・3 G。買った品のデータシートでピン配置を確認）"
+		(property "Description" "IF 増幅のカスコード下段（Q2 の代わり）。R5 は 47Ω に。N-Channel JFET 2SK192A（GR ランク、IDSS 6〜14mA。東芝 TO-92 小型 2-4E1D、1 D・2 S・3 G）"
 			(at 549.91 180.34 0)
 			(hide yes)

Commit message: L19 のタップを +9V 側から 2 回目 → 3 回目に（2SK192A-GR で下がった利得を戻す）
- L19 の値を T30-6 11T/3T に（L18 は 11T/2T のまま）。基板は変更なし（DRC 0・未配線 0・回路図との不一致 0、ERC 0）
- シミュレーション: RF 増幅 +7.7 → +10.5dB、前段の電力利得 +19.9dB・雑音指数 0.96dB、全体の雑音指数 1.3dB（混合器 NF 10dB）
- S9 で AD8307 の入力 −8.2dBm（J310 のときと同じ）なので、ファームウェアの RSSI_S9_MV 1900・AGC_TARGET_MV 1750 に戻す
- 部品表（L18・L19 を別の行に）、JLCPCB BOM・座標ファイル、README、調整手順、提出資料、部品実装図 PDF を更新

Co-Authored-By: Claude Opus 5.5 <noreply@anthropic.com>
Parts:
- L19: value T30-6 11T/2T -> T30-6 11T/3T
Changed lines of the file:
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@@
 			)
 		)
-		(property "Value" "T30-6 11T/2T"
+		(property "Value" "T30-6 11T/3T"
 			(at 276.86 125.73 0)
 			(show_name no)
@@
 			)
 		)
-		(property "Description" "RF 増幅の出力同調（ドレイン = 1 番、+9V = 3 番、タップ 2 番から混合器へ）"
+		(property "Description" "RF 増幅の出力同調（ドレイン = 1 番、+9V = 3 番、+9V 側から 3 回目のタップ 2 番から混合器へ）"
 			(at 271.78 119.38 0)
 			(hide yes)
